Commit message: Always create epick_extension link for stable URDF chain
Remove the conditional that skipped epick_extension when
extension_length=0. The link now always exists, ensuring a
stable link chain across all suction cup configurations.

When extension_length=0, the link sits at the body's top edge
with zero-size geometry — no visual or collision impact.

This allows MoveIt SRDF to reference epick_extension
unconditionally, avoiding link-not-found errors when switching
between cups with and without extensions.

File: epick_description/urdf/epick_single_suction_cup.xacro (robot description, xacro)
@@ -41,17 +41,14 @@
     <!-- inherits prefix, parent and origin_*, exposes body_link, body_length, body_color -->
     <xacro:epick_body parent="${parent}"/>
-    <xacro:property name="suction_cup_parent" value="${body_link}"/>
-    <xacro:property name="suction_cup_parent_length" value="${body_length}"/>
-    <!-- Extension (optional) -->
-    <xacro:if value="${extension_length * extension_radius > 0.0}">
-        <xacro:property name="suction_cup_parent" value="${prefix}epick_extension"/>
-        <xacro:property name="suction_cup_parent_length" value="${extension_length}"/>
-        <xacro:cylinder_link name="${prefix}epick_extension"
-                             radius="${extension_radius}"
-                             length="${extension_length}"
-                             color="${body_color}"
-                             parent="${body_link}"
-                             origin_xyz="0 0 ${(body_length + extension_length) / 2}"/>
-    </xacro:if>
+    <!-- Extension (always present for stable URDF link chain across cup configurations).
+         When extension_length=0, the link sits at the body's top edge with no geometry. -->
+    <xacro:cylinder_link name="${prefix}epick_extension"
+                         radius="${extension_radius}"
+                         length="${extension_length}"
+                         color="${body_color}"
+                         parent="${body_link}"
+                         origin_xyz="0 0 ${(body_length + extension_length) / 2}"/>
+    <xacro:property name="suction_cup_parent" value="${prefix}epick_extension"/>
+    <xacro:property name="suction_cup_parent_length" value="${extension_length}"/>
     <!-- Suction Cup -->
     <xacro:cylinder_link name="${prefix}epick_suction_cup"
